File: VfdController.kicad_pcb (KiCad board)
At the start: 2 copper layers, 100 x 58 mm, 30 parts, among them J1 Barrel_Jack_MountingPin, J2 Conn_02x13_Odd_Even, J3 CNT1230000, J4 VAL, J5 CNT1220000, J6 CNT1220000, U1 REG1220000, U2 ICS0020000, U3 ICS0020000

Commit message: Update remaining release docs.
Parts:
- removed G3: ~, 0-MRK:FTP-MRK-0003
- added J7: CNT1230000, 0-CNT:FTP-CNT-0008, F.Cu at (173.3, 125.2)
- added R4: 0, 0-RES:FTP-RES-0001, F.Cu at (163.6, 81.1)
- moved J2 30.5 mm to (103.7, 89.8), turned to 0 degrees
- moved C1 10.8 mm to (123.9, 108.8)
- moved C2 10.8 mm to (127.9, 108.8)
- moved C3 10.7 mm to (127.9, 90.4)
- moved C4 10.7 mm to (123.9, 90.4)
- moved J4 4.10 mm to (183.6, 101.5)
- moved J3 2.56 mm to (173.3, 131.6)
- turned U2 to 0 degrees
- turned U3 to 0 degrees
Connections:
- A1 pad 1: /pico_D7 -> /GPIO0
- A1 pad 10: /pico_D0 -> /GPIO7
- A1 pad 11: /pico_~{WR} -> /GPIO8
- A1 pad 12: /pico_A0 -> /GPIO9
- A1 pad 14: /pico_~{RD} -> /GPIO10
- A1 pad 15: /pico_SEL -> /GPIO11
- A1 pad 16: /pico_SER -> /GPIO12
- A1 pad 17: /pico_~{RESET} -> /GPIO13
- A1 pad 2: /pico_D6 -> /GPIO1
- A1 pad 21: unconnected-(A1-GPIO16-Pad21) -> /UART0_TX
- A1 pad 22: unconnected-(A1-GPIO17-Pad22) -> /UART0_RX
- A1 pad 4: /pico_D5 -> /GPIO2
- A1 pad 40: unconnected-(A1-VBUS-Pad40) -> Net-(A1-VBUS)
- A1 pad 5: /pico_D4 -> /GPIO3
- A1 pad 6: /pico_D3 -> /GPIO4
- A1 pad 7: /pico_D2 -> /GPIO5
- A1 pad 9: /pico_D1 -> /GPIO6
- U2 pad 1: +3V3 -> +5V
- U2 pad 10: GND -> unconnected-(U2-A7-Pad10)
- U2 pad 14: unconnected-(U2-B7-Pad14) -> GND
- U2 pad 15: unconnected-(U2-B6-Pad15) -> GND
- U2 pad 16: /~{WR} -> /GPIO13
- U2 pad 17: /A0 -> /GPIO12
- U2 pad 18: /~{RD} -> /GPIO11
- U2 pad 19: /SEL -> /GPIO10
- U2 pad 20: /SER -> /GPIO9
- U2 pad 21: /~{RESET} -> /GPIO8
- U2 pad 23: +5V -> +3V3
- U2 pad 24: +5V -> +3V3
- U2 pad 3: /pico_~{RESET} -> /D3
- U2 pad 4: /pico_SER -> /D4
- U2 pad 5: /pico_SEL -> /D5
- U2 pad 6: /pico_~{RD} -> /D6
- U2 pad 7: /pico_A0 -> /D7
- U2 pad 8: /pico_~{WR} -> /~{RESET}
- U2 pad 9: GND -> unconnected-(U2-A6-Pad9)
- U3 pad 1: +3V3 -> +5V
- U3 pad 10: /pico_D7 -> /D2
- U3 pad 14: /D7 -> /GPIO7
- U3 pad 15: /D6 -> /GPIO6
- U3 pad 16: /D5 -> /GPIO5
- U3 pad 17: /D4 -> /GPIO4
- U3 pad 18: /D3 -> /GPIO3
- U3 pad 19: /D2 -> /GPIO2
- U3 pad 20: /D1 -> /GPIO1
- U3 pad 21: /D0 -> /GPIO0
- U3 pad 23: +5V -> +3V3
- U3 pad 24: +5V -> +3V3
- U3 pad 3: /pico_D0 -> /SER
- U3 pad 4: /pico_D1 -> /SEL
- U3 pad 5: /pico_D2 -> /~{RD}
- U3 pad 6: /pico_D3 -> /A0
- U3 pad 7: /pico_D4 -> /~{WR}
- U3 pad 8: /pico_D5 -> /D0
- U3 pad 9: /pico_D6 -> /D1
Routing:
- net /GPIO0: track 0.00 -> 22.5 mm
- net /pico_D7: track 22.3 -> 0.00 mm
- net /GPIO1: track 0.00 -> 20.8 mm
- net /pico_D6: track 20.5 -> 0.00 mm
- net /pico_~{WR}: track 17.2 -> 0.00 mm
- net /GPIO8: track 0.00 -> 17.0 mm
- net /GPIO2: track 0.00 -> 16.8 mm
- net /pico_D0: track 16.7 -> 0.00 mm
- net /pico_D5: track 16.5 -> 0.00 mm
- net /UART0_TX: track 0.00 -> 16.3 mm
- net /GPIO7: track 0.00 -> 16.1 mm
- net /GPIO13: track 0.00 -> 16.0 mm
- net /pico_~{RESET}: track 15.7 -> 0.00 mm
- net /pico_A0: track 15.5 -> 0.00 mm
- net /pico_D1: track 15.1 -> 0.00 mm
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Other:
- board text added: "3700 ACM, VFD CONTROLLER - REV01"
- board text added: "RX"
- board text added: "TX"
- board text added: "VBUS"
- board text added: "VFD CONTROLLER REV01 30 AUG 2026"
- board text added: "VSYS"
- board text removed: "3700 ACM, VFD CONTROLLER - REV00"
- board text removed: "A0"
- board text removed: "D0"
- board text removed: "D1"
- board text removed: "D2"
- board text removed: "D3"
- board text removed: "D4"
- board text removed: "D5"
- board text removed: "D6"
- board text removed: "D7"
- board text removed: "SEL"
- board text removed: "SER"
- board text removed: "VFD CONTROLLER REV00 3 AUG 2026"
- board text removed: "~{RD}"
- board text removed: "~{WR}"
