File: VfdController.kicad_sch (KiCad schematic)
At the start: 12 parts, among them J1 Barrel_Jack_MountingPin, J2 Conn_02x13_Odd_Even, J3 CNT1130000, U3 ICS0020000, U4 ICS0020000

Commit message: Ordered REV00 PCB's x10
Parts:
- removed C5: 100n, 0-CAP:FTP-CAP-0001, symbol libdb:Capacitor/CAP-000-1042
- removed D1: DIO0999999, ~, symbol libdb:Diode/DIO-099-9999
- removed J3: CNT1130000, 0-CNT:FTP-CNT-0001, symbol libdb:Connector/CNT-113-0000
- removed U3, U4: ICS0020000, 1-PACKAGES:Generic-TSSOP-24_4.4x7.8mm_P0.65mm.kicad_mod, symbol libdb:IntegratedCircuit/ICS-002-0000
- added C10: 1u, 0-CAP:FTP-CAP-0001, symbol 00-JF:Capacitor/CAP-003-1051
- added C11, C12, C5, C6, C7, C8: 10u, 0-CAP:FTP-CAP-0002, symbol 00-JF:Capacitor/CAP-007-1061
- added C9: 100n, 0-CAP:FTP-CAP-0000, symbol 00-JF:Capacitor/CAP-001-1042
- added G1: ~, 0-MRK:FTP-MRK-0002b, symbol 00-JF:Marking/MRK-002-0000
- added G2: ~, 0-MRK:FTP-MRK-0000, symbol 00-JF:Marking/MRK-000-0000
- added G3: ~, 0-MRK:FTP-MRK-0003, symbol 00-JF:Marking/MRK-001-0000
- added J3: CNT1230000, 0-CNT:FTP-CNT-0008, symbol 00-JF:Connector/CNT-123-0000
- added J4: VAL, Connector_Molex:Molex_KK-396_A-41792-0006_1x06_P3.96mm_Horizontal, symbol 0-CNT:SYM-CNT-0008
- added J5, J6: CNT1220000, 0-CNT:FTP-CNT-0007, symbol 00-JF:Connector/CNT-122-0000
- added L1: 120Ω, 0-IND:FTP-IND-0002, symbol 00-JF:Magnetics/IND-203-1202
- added L2: 3.3u, 0-IND:FTP-IND-0000, symbol 00-JF:Magnetics/IND-002-3304
- added R1: 56k, 0-RES:FTP-RES-0001, symbol 00-JF:Resistor/RES-006-5604
- added R2: 10k, 0-RES:FTP-RES-0001, symbol 00-JF:Resistor/RES-006-1004
- added R3: 0, 0-RES:FTP-RES-0001, symbol 00-JF:Resistor/RES-000-0000
- added U1: REG1220000, 1-PACKAGES:Generic-SOT23-6, symbol 00-JF:Regulator/REG-122-0000
- added U2, U3: ICS0020000, 1-PACKAGES:Generic-TSSOP-24_4.4x7.8mm_P0.65mm, symbol 00-JF:IntegratedCircuit/ICS-002-0000
- J1: footprint (none) -> Connector_BarrelJack:BarrelJack_GCT_DCJ200-10-A_Horizontal
- J2: footprint (none) -> Connector_IDC:IDC-Header_2x13_P2.54mm_Vertical
Connections:
- net +3V3: now also C5.1, U2.1 (VCCA), U3.1 (VCCA)
- net +5V: now also C10.1, C11.1, C12.1, J4.1, L2.2, R1.1, R3.1, U2.23 (VCCB), U2.24 (VCCB), U3.23 (VCCB), U3.24 (VCCB); no longer A1.39 (VSYS)
- net A0: now also U2.17 (B4)
- net D0: now also U3.21 (B0)
- net D1: now also U3.20 (B1)
- net D2: now also U3.19 (B2)
- net D3: now also U3.18 (B3)
- net D4: now also U3.17 (B4)
- net D5: now also U3.16 (B5)
- net D6: now also U3.15 (B6)
- net D7: now also U3.14 (B7)
- net GND: now also C10.2, C11.2, C12.2, C5.2, C6.2, C7.2, C8.2, J3.2, J4.4, J5.2, J6.2, R2.2, U1.1 (GND), U2.10 (A7), U2.11 (GND), U2.12 (GND), U2.13 (GND), U2.2 (DIR), U2.22 (~{OE}), U2.9 (A6), U3.11 (GND), U3.12 (GND), U3.13 (GND), U3.2 (DIR), U3.22 (~{OE})
- net SEL: now also U2.19 (B2)
- net SER: now also U2.20 (B1)
- net VIN: now also C7.1, C8.1, L1.1, U1.3 (VIN), U1.5 (EN); no longer J1.1
- net pico_A0: now also A1.12 (GPIO9), U2.7 (A4)
- net pico_D0: now also A1.10 (GPIO7), U3.3 (A0)
- net pico_D1: now also A1.9 (GPIO6), U3.4 (A1)
- net pico_D2: now also A1.7 (GPIO5), U3.5 (A2)
- net pico_D3: now also A1.6 (GPIO4), U3.6 (A3)
- net pico_D4: now also A1.5 (GPIO3), U3.7 (A4)
- net pico_D5: now also A1.4 (GPIO2), U3.8 (A5)
- net pico_D6: now also A1.2 (GPIO1), U3.9 (A6)
- net pico_D7: now also A1.1 (GPIO0), U3.10 (A7)
- net pico_SEL: now also A1.15 (GPIO11), U2.5 (A2)
- net pico_SER: now also A1.16 (GPIO12), U2.4 (A1)
- net pico_~{RD}: now also A1.14 (GPIO10), U2.6 (A3)
- net pico_~{RESET}: now also A1.17 (GPIO13), U2.3 (A0)
- net pico_~{WR}: now also A1.11 (GPIO8), U2.8 (A5)
- net ~{RD}: now also U2.18 (B3)
- net ~{RESET}: now also J4.6, U2.21 (B0)
- net ~{WR}: now also U2.16 (B5)
- net clk: now reaches A1.D1 (SWCLK)
- net clk: now also J3.1
- net dio: now reaches A1.D3 (SWDIO)
- net dio: now also J3.3
- new net: A1.39 (VSYS), R3.2
- new net: C9.2, U1.6 (BST)
- new net jack: C6.1, J1.1, J5.1, J6.1, L1.2
- new net sw: C9.1, L2.1, U1.2 (SW)
- new net vfb: R1.2, R2.1, U1.4 (FB)
- no-connect marks 0 -> 20
Other:
- note added: "0.8V"
- note added: "5.28V [5.17V ... 5.39V]"
- note added: "DEBUG"
- note added: "DIR LOW - Bn Input, An Output DIR HI - An Input, Bn Output"
- note added: "TO AVOID SINKING CURRENT FROM USB 5V SET BUCK VOUT TO 5.25V"
- note added: "VIN [9... 12V]"
- note added: "~{OE} LOW - Output Enabled ~{OE} HI - Output HIZ"
- note removed: "VIN [5... 12V]"
- moved on the sheet: J1

Commit message: Update remaining release docs.
Parts:
- removed G3: ~, 0-MRK:FTP-MRK-0003, symbol 00-JF:Marking/MRK-001-0000
- added J7: CNT1230000, 0-CNT:FTP-CNT-0008, symbol 00-JF:Connector/CNT-123-0000
- added R4: 0, 0-RES:FTP-RES-0001, symbol 00-JF:Resistor/RES-000-0000
Connections:
- net +3V3: now also U2.23 (VCCB), U2.24 (VCCB), U3.23 (VCCB), U3.24 (VCCB); no longer U2.1 (VCCA), U3.1 (VCCA)
- net +5V: now also U2.1 (VCCA), U3.1 (VCCA), R4.1; no longer U2.23 (VCCB), U2.24 (VCCB), U3.23 (VCCB), U3.24 (VCCB)
- net A0: now also U3.6 (A3); no longer U2.17 (B4)
- net D0: now also U3.8 (A5); no longer U3.21 (B0)
- net D1: now also U3.9 (A6); no longer U3.20 (B1)
- net D2: now also U3.10 (A7); no longer U3.19 (B2)
- net D3: now also U2.3 (A0); no longer U3.18 (B3)
- net D4: now also U2.4 (A1); no longer U3.17 (B4)
- net D5: now also U2.5 (A2); no longer U3.16 (B5)
- net D6: now also U2.6 (A3); no longer U3.15 (B6)
- net D7: now also U2.7 (A4); no longer U3.14 (B7)
- net GND: now also U2.14 (B7), U2.15 (B6), J7.2; no longer U2.10 (A7), U2.9 (A6)
- net SEL: now also U3.4 (A1); no longer U2.19 (B2)
- net SER: now also U3.3 (A0); no longer U2.20 (B1)
- net ~{RD}: now also U3.5 (A2); no longer U2.18 (B3)
- net ~{RESET}: now also U2.8 (A5); no longer U2.21 (B0)
- net ~{WR}: now also U3.7 (A4); no longer U2.16 (B5)
- net UART0_TX: now reaches A1.21 (GPIO16)
- net UART0_TX: now also J7.1
- net UART0_RX: now reaches A1.22 (GPIO17)
- net UART0_RX: now also J7.3
- net at A1.40 (VBUS): now also R4.2
- net pico_A0 renamed GPIO9
- net GPIO9: now also U2.20 (B1); no longer U2.7 (A4)
- net pico_D0 renamed GPIO7
- net GPIO7: now also U3.14 (B7); no longer U3.3 (A0)
- net pico_D1 renamed GPIO6
- net GPIO6: now also U3.15 (B6); no longer U3.4 (A1)
- net pico_D2 renamed GPIO5
- net GPIO5: now also U3.16 (B5); no longer U3.5 (A2)
- net pico_D3 renamed GPIO4
- net GPIO4: now also U3.17 (B4); no longer U3.6 (A3)
- net pico_D4 renamed GPIO3
- net GPIO3: now also U3.18 (B3); no longer U3.7 (A4)
- net pico_D5 renamed GPIO2
- net GPIO2: now also U3.19 (B2); no longer U3.8 (A5)
- net pico_D6 renamed GPIO1
- net GPIO1: now also U3.20 (B1); no longer U3.9 (A6)
- net pico_D7 renamed GPIO0
- net GPIO0: now also U3.21 (B0); no longer U3.10 (A7)
- net pico_SEL renamed GPIO11
- net GPIO11: now also U2.18 (B3); no longer U2.5 (A2)
- net pico_SER renamed GPIO12
- net GPIO12: now also U2.17 (B4); no longer U2.4 (A1)
- net pico_~{RD} renamed GPIO10
- net GPIO10: now also U2.19 (B2); no longer U2.6 (A3)
- net pico_~{RESET} renamed GPIO13
- net GPIO13: now also U2.16 (B5); no longer U2.3 (A0)
- net pico_~{WR} renamed GPIO8
- net GPIO8: now also U2.21 (B0); no longer U2.8 (A5)
- no-connect marks 20 -> 18
Other:
- note added: "PROG"
- note added: "UART0"
- note added: "VCCA = [4.5V... 5.5V] VCCB = [2.7V... 3.6V]"
- note removed: "DEBUG"
- moved on the sheet: R3
